Commit message: ros2 moveit tx200

File: staubli_tx200_support/urdf/tx200_macro.xacro (robot description, xacro)
@@ -169,17 +169,17 @@
     </joint>
     <!-- ROS-Industrial 'flange' frame: attachment point for EEF models -->
-    <link name="${prefix}flange" />
+    <!-- <link name="${prefix}flange" />
     <joint name="${prefix}joint_6-flange" type="fixed">
       <origin xyz="0 0 0" rpy="0 ${radians(-90.0)} 0" />
       <parent link="${prefix}link_6" />
       <child link="${prefix}flange" />
-    </joint>
+    </joint> -->
     <!-- ROS-Industrial 'tool0' frame: all-zeros tool frame -->
-    <link name="${prefix}tool0" />
+    <!-- <link name="${prefix}tool0" />
     <joint name="${prefix}flange-tool0" type="fixed">
       <origin xyz="0 0 0" rpy="0 ${radians(90.0)} 0" />
       <parent link="${prefix}flange" />
       <child link="${prefix}tool0" />
-    </joint>
+    </joint> -->
   </xacro:macro>
 </robot>

Commit message: colcon ignores

File: staubli_tx200_support/urdf/tx200_macro.xacro (robot description, xacro)
@@ -4,5 +4,5 @@
   <xacro:macro name="staubli_tx200" params="prefix">
     <!-- links: main serial chain -->
-    <link name="${prefix}base_link">
+    <link name="${prefix}base">
       <visual>
         <origin xyz="0 0 0" rpy="0 0 0"/>
@@ -112,5 +112,5 @@
     <joint name="${prefix}joint_1" type="revolute">
       <origin xyz="0 0 0" rpy="0 0 0"/>
-      <parent link="${prefix}base_link"/>
+      <parent link="${prefix}base"/>
       <child link="${prefix}link_1"/>
       <axis xyz="0 0 1"/>
@@ -162,24 +162,17 @@
     </joint>
     <!-- ROS-Industrial 'base' frame: base_link to Staubli World Coordinates transform -->
-    <link name="${prefix}base" />
+    <link name="${prefix}base_link" />
     <joint name="${prefix}base_link-base" type="fixed">
-      <origin xyz="0 0 -0.642" rpy="0 0 0"/>
+      <origin xyz="0 0 0.642" rpy="0 0 0"/>
       <parent link="${prefix}base_link"/>
       <child link="${prefix}base"/>
     </joint>
     <!-- ROS-Industrial 'flange' frame: attachment point for EEF models -->
-    <!-- <link name="${prefix}flange" />
+    <link name="${prefix}flange" />
     <joint name="${prefix}joint_6-flange" type="fixed">
-      <origin xyz="0 0 0" rpy="0 ${radians(-90.0)} 0" />
+      <origin xyz="0 0 0" rpy="0 0 0" />
       <parent link="${prefix}link_6" />
       <child link="${prefix}flange" />
-    </joint> -->
-    <!-- ROS-Industrial 'tool0' frame: all-zeros tool frame -->
-    <!-- <link name="${prefix}tool0" />
-    <joint name="${prefix}flange-tool0" type="fixed">
-      <origin xyz="0 0 0" rpy="0 ${radians(90.0)} 0" />
-      <parent link="${prefix}flange" />
-      <child link="${prefix}tool0" />
-    </joint> -->
+    </joint>
   </xacro:macro>
 </robot>
